File: HbridgeS_UNIT.kicad_pcb (KiCad board)
At the start: 2 copper layers, 20.6 x 28 mm, 7 parts, among them CN1 CON_GROVE, J2 Conn_01x04, U1 DRV_RZ7899

Commit message: add PCB data
Parts:
- moved C3 11.3 mm to (16.7, 11.8), turned to -90 degrees
- moved JP1 9.21 mm to (16.5, 11.8)
- moved C2 6.11 mm to (13.3, 11.0), turned to -90 degrees
- moved C1 6.02 mm to (14.8, 11.0), turned to -90 degrees
- moved U1 5.20 mm to (8.80, 12.1), turned to 180 degrees
Connections:
- J2 pad 1: /OUT_P -> GND
- J2 pad 2: /OUT_N -> VDD
- J2 pad 3: VDD -> /OUT_P
- J2 pad 4: GND -> /OUT_N
Routing:
- net /MR: track 18.7 -> 10.6 mm
- net +5V: track 13.5 -> 19.1 mm, vias 1 -> 0
- net /OUT_P: track 10.2 -> 5.41 mm, vias 8 -> 27
- net GND: track 26.4 -> 28.4 mm
- net /OUT_N: track 6.58 -> 8.15 mm, vias 28 -> 19
- net VD: track 6.88 -> 7.56 mm
